Commit message: Update for Gazebo simulation
roslaunch Ball_bot ball_bot.launch to start the simulation.
rosrun turtlebot3_teleop turtlebot3_teleop_key can be used for driving.

File: urdf/ball_bot.gazebo.xacro (robot description, xacro)
@@ -5,9 +5,11 @@
   <xacro:arg name="imu_visual"    default="false"/>
   <gazebo reference="base_link">
+    <mu1>0.1</mu1>
+    <mu2>0.1</mu2>
     <material>Gazebo/White</material>
   </gazebo>
   <gazebo reference="wheel_left_link">
-    <mu1>0.1</mu1>
-    <mu2>0.1</mu2>
+    <mu1>0.8</mu1>
+    <mu2>0.8</mu2>
     <kp>500000.0</kp>
     <kd>10.0</kd>
@@ -18,6 +20,6 @@
   </gazebo>
   <gazebo reference="wheel_right_link">
-    <mu1>0.1</mu1>
-    <mu2>0.1</mu2>
+    <mu1>0.8</mu1>
+    <mu2>0.8</mu2>
     <kp>500000.0</kp>
     <kd>10.0</kd>

File: urdf/ball_bot.urdf.xacro (robot description, xacro)
@@ -7,9 +7,9 @@
     <parent link="base_footprint"/>
     <child link="base_link" />
-    <origin xyz="0 0 0.010" rpy="0 0 0"/>
+    <origin xyz="0 0 0" rpy="0 0 0"/>
   </joint>
   <link name="base_link">
     <visual>
-      <origin xyz="0 0 0" rpy="1.57 0 0"/>
+      <origin xyz="0 0.11 -0.0055" rpy="1.57 0 0"/>
       <geometry>
         <mesh filename="package://Ball_bot/meshes/base.stl" scale="0.001 0.001 0.001"/>
@@ -18,5 +18,5 @@
     </visual>
     <collision>
-      <origin xyz="0 0 0" rpy="1.57 0 0"/>
+      <origin xyz="0 0.11 -0.0055" rpy="1.57 0 0"/>
       <geometry>
         <mesh filename="package://Ball_bot/meshes/base.stl" scale="0.001 0.001 0.001"/>
@@ -24,6 +24,6 @@
     </collision>
     <inertial>
-      <origin xyz="0.0 -0.05 -0.01" rpy="0 0 0"/>
-      <mass value="1.3729096e+00"/>
+      <origin xyz="0.0 0.05 -0.04" rpy="0 0 0"/>
+      <mass value="0.8"/>
       <inertia ixx="8.7002718e-03" ixy="-4.7576583e-05" ixz="1.1160499e-04"
                iyy="8.6195418e-03" iyz="-3.5422299e-06"
@@ -34,29 +34,57 @@
     <parent link="base_link"/>
     <child link="wheel_left_link"/>
-    <origin xyz="0 0 0" rpy="-1.57 0 0"/>
+    <origin xyz="-0.025706 0 0" rpy="0 0 0"/>
     <axis xyz="1 0 0"/>
   </joint>
   <link name="wheel_left_link">
     <visual>
-      <origin xyz="0 0 0" rpy="1.57 0 1.57"/>
-      <geometry>
-        <mesh filename="package://Ball_bot/meshes/wheel.stl" scale="0.001 0.001 0.001"/>
-      </geometry>
-      <material name="dark"/>
-    </visual>
-    <collision>
-      <origin xyz="0 0 0" rpy="1.57 0 1.57"/>
-      <geometry>
-        <mesh filename="package://Ball_bot/meshes/wheel.stl" scale="0.001 0.001 0.001"/>
-      </geometry>
-    </collision>
-    <inertial>
-      <origin xyz="0 0 0" />
-      <mass value="2.8498940e-02" />
-      <inertia ixx="1.1175580e-05" ixy="-4.2369783e-11" ixz="-5.9381719e-09"
-               iyy="1.1192413e-05" iyz="-1.4400107e-11"
-               izz="2.0712558e-05" />
-      </inertial>
-  </link>
+      <origin xyz="-0.014775 0 -0.069411" rpy="0 0 0"/>
+      <geometry>
+        <mesh filename="package://Ball_bot/meshes/wheel.stl" scale="0.001 0.001 0.001"/>
+      </geometry>
+      <material name="dark"/>
+    </visual>
+    <collision>
+      <origin xyz="-0.014775 0 -0.069411" rpy="0 0 0"/>
+      <geometry>
+        <mesh filename="package://Ball_bot/meshes/wheel.stl" scale="0.001 0.001 0.001"/>
+      </geometry>
+    </collision>
+    <inertial>
+      <origin xyz="0 0 0" />
+      <mass value="2.8498940e-02" />
+      <inertia ixx="1.1175580e-05" ixy="-4.2369783e-11" ixz="-5.9381719e-09"
+               iyy="1.1192413e-05" iyz="-1.4400107e-11"
+               izz="2.0712558e-05" />
+      </inertial>
+  </link>
+  <joint name="wheel_right_joint" type="continuous">
+    <parent link="base_link"/>
+    <child link="wheel_right_link"/>
+    <origin xyz="0.025706 0 0" rpy="0 0 3.14"/>
+    <axis xyz="-1 0 0"/>
+  </joint>
+  <link name="wheel_right_link">
+    <visual>
+      <origin xyz="-0.014775 0 -0.069411" rpy="0 0 0"/>
+      <geometry>
+        <mesh filename="package://Ball_bot/meshes/wheel.stl" scale="0.001 0.001 0.001"/>
+      </geometry>
+      <material name="dark"/>
+    </visual>
+    <collision>
+      <origin xyz="-0.014775 0 -0.069411" rpy="0 0 0"/>
+      <geometry>
+        <mesh filename="package://Ball_bot/meshes/wheel.stl" scale="0.001 0.001 0.001"/>
+      </geometry>
+    </collision>
+    <inertial>
+      <origin xyz="0 0 0" />
+      <mass value="2.8498940e-02" />
+      <inertia ixx="1.1175580e-05" ixy="-4.2369783e-11" ixz="-5.9381719e-09"
+               iyy="1.1192413e-05" iyz="-1.4400107e-11"
+               izz="2.0712558e-05" />
+      </inertial>
+  </link> -->
 <!--
   <joint name="wheel_left_joint" type="continuous">

Commit message: update for camera

File: urdf/ball_bot.gazebo.xacro (robot description, xacro)
@@ -119,46 +119,46 @@
   </gazebo>
 <!--link : https://www.raspberrypi.org/documentation/hardware/camera/-->
-  <gazebo reference="camera_rgb_frame">
-    <sensor name="camera" type="depth">
-      <update_rate>20</update_rate>
-      <camera>
-        <horizontal_fov>1.349721</horizontal_fov>
-        <image>
-          <width>640</width>
-          <height>480</height>
-          <format>R8G8B8</format>
-        </image>
-        <clip>
-          <near>0.05</near>
-          <far>12.0</far>
-        </clip>
-      </camera>
-      <plugin name="camera_plugin" filename="libgazebo_ros_openni_kinect.so">
-        <baseline>0.2</baseline>
-        <alwaysOn>true</alwaysOn>
-        <!-- Keep this zero, update_rate in the parent <sensor> tag
-          will control the frame rate. -->
-        <updateRate>0.0</updateRate>
-        <cameraName>camera_ir</cameraName>
-        <imageTopicName>/camera/color/image_raw</imageTopicName>
-        <cameraInfoTopicName>/camera/color/camera_info</cameraInfoTopicName>
-        <depthImageTopicName>/camera/depth/image_raw</depthImageTopicName>
-        <depthImageCameraInfoTopicName>/camera/depth/camera_info</depthImageCameraInfoTopicName>
-        <pointCloudTopicName>/camera/depth/points</pointCloudTopicName>
-        <frameName>base_footprint</frameName>
-        <pointCloudCutoff>0.105</pointCloudCutoff>
-        <pointCloudCutoffMax>12.0</pointCloudCutoffMax>
-        <distortionK1>0</distortionK1>
-        <distortionK2>0</distortionK2>
-        <distortionK3>0</distortionK3>
-        <distortionT1>0</distortionT1>
-        <distortionT2>0</distortionT2>
-        <CxPrime>0</CxPrime>
-        <Cx>0</Cx>
-        <Cy>0</Cy>
-        <focalLength>0</focalLength>
-        <hackBaseline>0</hackBaseline>
-      </plugin>
-    </sensor>
-  </gazebo>
+<gazebo reference="camera_rgb_frame">
+  <sensor name="camera" type="depth">
+    <update_rate>20</update_rate>
+    <camera>
+      <horizontal_fov>1.349721</horizontal_fov>
+      <image>
+        <width>640</width>
+        <height>480</height>
+        <format>R8G8B8</format>
+      </image>
+      <clip>
+        <near>0.05</near>
+        <far>12.0</far>
+      </clip>
+    </camera>
+    <plugin name="camera_plugin" filename="libgazebo_ros_openni_kinect.so">
+      <baseline>0.2</baseline>
+      <alwaysOn>true</alwaysOn>
+      <!-- Keep this zero, update_rate in the parent <sensor> tag
+        will control the frame rate. -->
+      <updateRate>0.0</updateRate>
+      <cameraName>camera_ir</cameraName>
+      <imageTopicName>/camera/color/image_raw</imageTopicName>
+      <cameraInfoTopicName>/camera/color/camera_info</cameraInfoTopicName>
+      <depthImageTopicName>/camera/depth/image_raw</depthImageTopicName>
+      <depthImageCameraInfoTopicName>/camera/depth/camera_info</depthImageCameraInfoTopicName>
+      <pointCloudTopicName>/camera/depth/points</pointCloudTopicName>
+      <frameName>base_footprint</frameName>
+      <pointCloudCutoff>0.105</pointCloudCutoff>
+      <pointCloudCutoffMax>12.0</pointCloudCutoffMax>
+      <distortionK1>0</distortionK1>
+      <distortionK2>0</distortionK2>
+      <distortionK3>0</distortionK3>
+      <distortionT1>0</distortionT1>
+      <distortionT2>0</distortionT2>
+      <CxPrime>0</CxPrime>
+      <Cx>0</Cx>
+      <Cy>0</Cy>
+      <focalLength>0</focalLength>
+      <hackBaseline>0</hackBaseline>
+    </plugin>
+  </sensor>
+</gazebo>
 </robot>

File: urdf/ball_bot.urdf.xacro (robot description, xacro)
@@ -87,89 +87,6 @@
       </inertial>
   </link> -->
-<!--
-  <joint name="wheel_left_joint" type="continuous">
-    <parent link="base_link"/>
-    <child link="wheel_left_link"/>
-    <origin xyz="0 0 0" rpy="-1.57 0 0"/>
-    <axis xyz="0 0 1"/>
-  </joint>
-  <link name="wheel_left_link">
-    <visual>
-      <origin xyz="0 0 0" rpy="1.57 0 0"/>
-      <geometry>
-        <mesh filename="package://Ball_bot/meshes/wheel.stl" scale="0.001 0.001 0.001"/>
-      </geometry>
-      <material name="dark"/>
-    </visual>
-    <collision>
-      <origin xyz="0 0 0" rpy="0 0 0"/>
-      <geometry>
-        <mesh filename="package://Ball_bot/meshes/wheel.stl" scale="0.001 0.001 0.001"/>
-      </geometry>
-    </collision>
-    <inertial>
-      <origin xyz="0 0 0" />
-      <mass value="2.8498940e-02" />
-      <inertia ixx="1.1175580e-05" ixy="-4.2369783e-11" ixz="-5.9381719e-09"
-               iyy="1.1192413e-05" iyz="-1.4400107e-11"
-               izz="2.0712558e-05" />
-      </inertial>
-  </link>
-  <joint name="wheel_right_joint" type="continuous">
-    <parent link="base_link"/>
-    <child link="wheel_right_link"/>
-    <origin xyz="0.0 -0.144 0.023" rpy="-1.57 0 0"/>
-    <axis xyz="0 0 1"/>
-  </joint>
-  <link name="wheel_right_link">
-    <visual>
-      <origin xyz="0 0 0" rpy="1.57 0 0"/>
-      <geometry>
-        <mesh filename="package://Ball_bot/meshes/wheel.stl" scale="0.001 0.001 0.001"/>
-      </geometry>
-      <material name="dark"/>
-    </visual>
-    <collision>
-      <origin xyz="0 0 0" rpy="0 0 0"/>
-      <geometry>
-        <mesh filename="package://Ball_bot/meshes/wheel.stl" scale="0.001 0.001 0.001"/>
-      </geometry>
-    </collision>
-    <inertial>
-      <origin xyz="0 0 0" />
-      <mass value="2.8498940e-02" />
-      <inertia ixx="1.1175580e-05" ixy="-4.2369783e-11" ixz="-5.9381719e-09"
-               iyy="1.1192413e-05" iyz="-1.4400107e-11"
-               izz="2.0712558e-05" />
-      </inertial>
-  </link> -->
-  <!-- <joint name="imu_joint" type="fixed">
-    <parent link="base_link"/>
-    <child link="imu_link"/>
-    <origin xyz="0.0 0 0.068" rpy="0 0 0"/>
-  </joint>
-  <link name="imu_link"/>
-  <joint name="scan_joint" type="fixed">
-    <parent link="base_link"/>
-    <child link="base_scan"/>
-    <origin xyz="-0.064 0 0.122" rpy="0 0 0"/>
-  </joint>
-  <link name="base_scan">
-    <collision>
-      <origin xyz="0.015 0 -0.0065" rpy="0 0 0"/>
-      <geometry>
-        <cylinder length="0.0315" radius="0.055"/>
-      </geometry>
-    </collision>
-    <inertial>
-      <mass value="0.114" />
-      <origin xyz="0 0 0" />
-      <inertia ixx="0.001" ixy="0.0" ixz="0.0"
-               iyy="0.001" iyz="0.0"
-               izz="0.001" />
-    </inertial>
-  </link>
   <joint name="camera_joint" type="fixed">
-    <origin xyz="0.073 -0.011 0.107" rpy="0 0 0"/>
+    <origin xyz="0.073 -0.011 0.107" rpy="0 0 -1.57"/>
     <parent link="base_link"/>
     <child link="camera_link"/>
@@ -189,16 +106,10 @@
   </joint>
   <link name="camera_rgb_frame">
-    <visual>
-      <origin xyz="0 0 -0.01" rpy="-1.57 0 -1.57"/>
-      <geometry>
-        <mesh filename="package://Ball_bot/meshes/sensors/d435.dae" scale="1 1 1"/>
-      </geometry>
-    </visual>
   </link>
   <joint name="camera_rgb_optical_joint" type="fixed">
-    <origin xyz="0 0 0" rpy="-1.57 0 -1.57"/>
+    <origin xyz="0 0 0" rpy="0 0 0"/>
     <parent link="camera_rgb_frame"/>
     <child link="camera_rgb_optical_frame"/>
   </joint>
-  <link name="camera_rgb_optical_frame"/> -->
+  <link name="camera_rgb_optical_frame"/>
 </robot>

Commit message: new world environments

File: urdf/ball_bot.gazebo.xacro (robot description, xacro)
@@ -7,5 +7,5 @@
     <mu1>0.1</mu1>
     <mu2>0.1</mu2>
-    <material>Gazebo/White</material>
+    <material>Gazebo/Grey</material>
   </gazebo>
   <gazebo reference="wheel_left_link">

File: urdf/ball_bot.urdf.xacro (robot description, xacro)
@@ -15,5 +15,5 @@
         <mesh filename="package://Ball_bot/meshes/base.stl" scale="0.001 0.001 0.001"/>
       </geometry>
-      <material name="white"/>
+      <material name="grey"/>
     </visual>
     <collision>
